Commit message: Added ft sensors frames and in simulation

File: walkman_urdf/urdf/gazebo/force_torque.gazebo.xacro (robot description, xacro)
@@ -31,3 +31,27 @@
 		</sensor>
 	</gazebo>
+	<gazebo reference="LWrj2">
+		<sensor type="force_torque" name="l_arm_ft">
+                     <force_torque>
+                       <frame>sensor</frame>
+                       <measure_direction>child_to_parent</measure_direction>
+                     </force_torque>
+			<always_on>true</always_on>
+			<visualize>true</visualize>
+			<update_rate>1000</update_rate>
+			<pose>0.0 0.0 -0.0235 0 0 0</pose>
+		</sensor>
+	</gazebo>
+	<gazebo reference="RWrj2">
+		<sensor type="force_torque" name="r_arm_ft">
+                     <force_torque>
+                       <frame>sensor</frame>
+                       <measure_direction>child_to_parent</measure_direction>
+                     </force_torque>
+			<always_on>true</always_on>
+			<visualize>true</visualize>
+			<update_rate>1000</update_rate>
+			<pose>0.0 0.0 -0.0235 0 0 0</pose>
+		</sensor>
+	</gazebo>
 </robot>

File: walkman_urdf/urdf/walkman.urdf.xacro (robot description, xacro)
@@ -32,4 +32,16 @@
     <origin xyz="0.005 0 -0.107" rpy="0 0 0"/>
 </joint>
+<link name="l_arm_ft"/>
+<link name="r_arm_ft"/>
+<joint name="l_arm_ft_joint" type="fixed">
+    <parent link="LWrMot3"/>
+    <child link="l_arm_ft"/>
+    <origin xyz="0 0 ${-23.5*mmTom}" rpy="0 0 0" />
+</joint>
+<joint name="r_arm_ft_joint" type="fixed">
+    <parent link="RWrMot3"/>
+    <child link="r_arm_ft"/>
+    <origin xyz="0 0 ${-23.5*mmTom}" rpy="0 0 0" />
+</joint>
 <xacro:include filename="$(find walkman_urdf)/urdf/sensors/imu.urdf.xacro"/>
 </robot>

File: walkman_urdf/urdf/walkman_base.urdf.xacro (robot description, xacro)
@@ -120,17 +120,3 @@
 </joint>
 <xacro:include filename="$(find walkman_urdf)/urdf/parts/soft_hand.urdf.xacro" />
-<!--
-<link name="l_arm_ft"/>
-	<link name="r_arm_ft"/>
-	<joint name="l_arm_ft_joint" type="fixed">
-	    <parent link="LWrMot3"/>
-	    <child link="l_arm_ft"/>
-	    <origin xyz="0 0 -0.0565" rpy="0 0 0" />
-	</joint>
-	<joint name="r_arm_ft_joint" type="fixed">
-	    <parent link="RWrMot3"/>
-	    <child link="r_arm_ft"/>
-	    <origin xyz="0 0 -0.0565" rpy="0 0 0" />
-	</joint>
--->
 </robot>
