Commit message: Updated joint limits

File: walkman_urdf/urdf/parts/arms.urdf.xacro (robot description, xacro)
@@ -4,4 +4,5 @@
 <xacro:property name="mmTom" value="0.001" />
 <xacro:property name="mm2Tom2" value="${0.001*0.001}" />
+<xacro:property name="DEG2RAD" value="${PI/180.}" />
 <!-- RIGHT ARM -->
 <link name ="RShp">
@@ -150,5 +151,5 @@
     <origin xyz="${45.7475*mmTom} ${-169.137*mmTom} ${155.126*mmTom}" rpy="-0.174533 0 0.5235988" />
     <axis xyz="0 1 0" />
-    <limit velocity="6.283" effort="120" lower="${-PI}" upper="${PI}" />
+    <limit velocity="6.283" effort="147" lower="${-195.*DEG2RAD}" upper="${95.*DEG2RAD}" />
     <dynamics friction="0" damping="3.0"/>
 </joint>
@@ -158,5 +159,5 @@
     <origin xyz="${-90.15*mmTom} ${-62*mmTom} 0" rpy="0.1745327 0 0" />
     <axis xyz="1 0 0" />
-    <limit velocity="6.283" effort="120" lower="${-PI}" upper="${PI}" />
+    <limit velocity="6.283" effort="120" lower="${-200.*DEG2RAD}" upper="0" />
     <dynamics friction="0" damping="3.0"/>
 </joint>
@@ -166,5 +167,5 @@
     <origin xyz="${90.15*mmTom} 0 ${-218.15*mmTom}" rpy="0 0 0" />
     <axis xyz="0 0 1" />
-    <limit velocity="6.283" effort="120" lower="${-PI}" upper="${PI}" />
+    <limit velocity="6.283" effort="147" lower="${-150.*DEG2RAD}" upper="${150.*DEG2RAD}" />
     <dynamics friction="0" damping="3.0"/>
 </joint>
@@ -174,5 +175,5 @@
     <origin xyz="${45.*mmTom} ${-55.15*mmTom} ${-74.*mmTom}" rpy="0 0 0" />
     <axis xyz="0 1 0" />
-    <limit velocity="6.283" effort="120" lower="${-170.0*toRad}" upper="${34.0*toRad}" />
+    <limit velocity="6.283" effort="147" lower="${-170.0*toRad}" upper="${34.0*toRad}" />
     <dynamics friction="0" damping="3.0"/>
 </joint>
@@ -182,5 +183,5 @@
     <origin xyz="${-15.*mmTom} ${55.15*mmTom} ${-95.*mmTom}" rpy="0 0 0"/>
     <axis xyz="0 0 1" />
-    <limit velocity="6.283" effort="60" lower="-2.529" upper="2.529" />
+    <limit velocity="6.283" effort="55" lower="${-150*DEG2RAD}" upper="${150*DEG2RAD}" />
     <dynamics friction="0" damping="0.03"/>
 </joint>
@@ -190,5 +191,5 @@
     <origin xyz="0 ${-49*mmTom} ${-156.*mmTom}" rpy="0 0 0"/>
     <axis xyz="0 1 0"/>
-    <limit velocity="6.283" effort="60" lower="-1.48" upper="1.48" />
+    <limit velocity="6.283" effort="55" lower="${-90.*DEG2RAD}" upper="${90.*DEG2RAD}" />
     <dynamics friction="0" damping="0.03"/>
 </joint>
@@ -198,5 +199,5 @@
        <origin xyz="0 ${49*mmTom} ${-174.*mmTom}" rpy="0 0 0"/>
        <axis xyz="0 0 1"/>
-       <limit velocity="6.283" effort="60" lower="-1.48" upper="1.48" />
+       <limit velocity="6.283" effort="27" lower="${-150.*DEG2RAD}" upper="${150.*DEG2RAD}" />
        <dynamics friction="0" damping="0.03"/>
 </joint>
@@ -347,5 +348,5 @@
     <origin xyz="${45.7475*mmTom} ${169.137*mmTom} ${155.126*mmTom}" rpy="0.174533 0 -0.5235988" />
     <axis xyz="0 1 0" />
-    <limit velocity="6.283" effort="120" lower="${-PI}" upper="${PI}" />
+    <limit velocity="6.283" effort="147" lower="${-195.*DEG2RAD}" upper="${95.*DEG2RAD}" />
     <dynamics friction="0" damping="3.0"/>
 </joint>
@@ -355,5 +356,5 @@
     <origin xyz="${-90.15*mmTom} ${62*mmTom} 0" rpy="-0.1745327 0 0" />
     <axis xyz="1 0 0" />
-    <limit velocity="6.283" effort="120" lower="${-PI}" upper="${PI}" />
+    <limit velocity="6.283" effort="120" lower="0" upper="${200.*DEG2RAD}" />
     <dynamics friction="0" damping="3.0"/>
 </joint>
@@ -363,5 +364,5 @@
     <origin xyz="${90.15*mmTom} 0 ${-218.15*mmTom}" rpy="0 0 0" />
     <axis xyz="0 0 1" />
-    <limit velocity="6.283" effort="120" lower="${-PI}" upper="${PI}" />
+    <limit velocity="6.283" effort="147" lower="${-150.*DEG2RAD}" upper="${150.*DEG2RAD}" />
     <dynamics friction="0" damping="3.0"/>
 </joint>
@@ -371,5 +372,5 @@
     <origin xyz="${45.*mmTom} ${55.15*mmTom} ${-74.*mmTom}" rpy="0 0 0" />
     <axis xyz="0 1 0" />
-    <limit velocity="6.283" effort="120" lower="${-170.0*toRad}" upper="${34.0*toRad}" />
+    <limit velocity="6.283" effort="147" lower="${-145.0*DEG2RAD}" upper="${20.0*DEG2RAD}" />
     <dynamics friction="0" damping="3.0"/>
 </joint>
@@ -379,5 +380,5 @@
     <origin xyz="${-15.*mmTom} ${-55.15*mmTom} ${-95.*mmTom}" rpy="0 0 0"/>
     <axis xyz="0 0 1" />
-    <limit velocity="6.283" effort="60" lower="-2.529" upper="2.529" />
+    <limit velocity="6.283" effort="55" lower="${-150.0*DEG2RAD}" upper="${150.0*DEG2RAD}" />
     <dynamics friction="0" damping="0.03"/>
 </joint>
@@ -387,5 +388,5 @@
     <origin xyz="0 ${49*mmTom} ${-156.*mmTom}" rpy="0 0 0"/>
     <axis xyz="0 1 0"/>
-    <limit velocity="6.283" effort="60" lower="-1.48" upper="1.48" />
+    <limit velocity="6.283" effort="55" lower="${-90.0*DEG2RAD}" upper="${90.0*DEG2RAD}" />
     <dynamics friction="0" damping="0.03"/>
 </joint>
@@ -395,5 +396,5 @@
        <origin xyz="0 ${-49*mmTom} ${-174.*mmTom}" rpy="0 0 0"/>
        <axis xyz="0 0 1"/>
-       <limit velocity="6.283" effort="60" lower="-1.48" upper="1.48" />
+       <limit velocity="6.283" effort="27" lower="${-150.0*DEG2RAD}" upper="${150.0*DEG2RAD}" />
        <dynamics friction="0" damping="0.03"/>
 </joint>

File: walkman_urdf/urdf/parts/legs.urdf.xacro (robot description, xacro)
@@ -6,4 +6,5 @@
 <xacro:property name="PI" value="3.14159265359" />
 <xacro:property name="PI_2" value="1.57079632679" />
+<xacro:property name="DEG2RAD" value="${PI/180.0}" />
 <!-- LINKS -->
 <!-- ********************RIGHT LEG******************** -->
@@ -256,5 +257,5 @@
     <origin xyz="${156.9*mmTom} ${-60.*mmTom} ${-108.*mmTom}" rpy="0 0 0" />
     <axis xyz="1 0 0" />
-    <limit velocity="6.283" effort="400" lower="-0.87222" upper="0.697778" />
+    <limit velocity="6.283" effort="400" lower="${-50.*DEG2RAD}" upper="${40.*DEG2RAD}" />
     <dynamics friction="0" damping="3.0"/>
   </joint>
@@ -264,5 +265,5 @@
     <origin xyz="-0.0889 -0.121032 -0.217872" rpy="0 0 0" />
     <axis xyz="0 0 1" />
-    <limit velocity="6.283" effort="140" lower="-1.57" upper="0.872222" />
+    <limit velocity="6.283" effort="140" lower="${-90.*DEG2RAD}" upper="${50.*DEG2RAD}" />
     <dynamics friction="0" damping="3.0"/>
   </joint>
@@ -272,5 +273,5 @@
     <origin xyz="0.0 0.0 0.0" rpy="0 0 0" />
     <axis xyz="0 1 0" />
-    <limit velocity="6.283" effort="400" lower="-2.09333" upper="1.046667" />
+    <limit velocity="6.283" effort="400" lower="${-120.*DEG2RAD}" upper="${60.*DEG2RAD}" />
     <dynamics friction="0" damping="3.0"/>
   </joint>
@@ -280,5 +281,5 @@
     <origin xyz="0.0 0.0 -0.356" rpy="0 0 0" />
     <axis xyz="0 1 0" />
-    <limit velocity="6.283" effort="400" lower="0.0" upper="2.442222" />
+    <limit velocity="6.283" effort="400" lower="0.0" upper="${140.*DEG2RAD}" />
     <dynamics friction="0" damping="3.0"/>
   </joint>
@@ -288,5 +289,5 @@
     <origin xyz="0.0 0.0 -0.4" rpy="0 0 0" />
     <axis xyz="0 1 0" />
-    <limit velocity="6.283" effort="330" lower="-1.39556" upper="0.697778" />
+    <limit velocity="6.283" effort="330" lower="${-80.*DEG2RAD}" upper="${40.*DEG2RAD}" />
     <dynamics friction="0" damping="3.0"/>
   </joint>
@@ -296,5 +297,5 @@
       <origin xyz="0.0 0.0 0.0" rpy="0 0 0" />
       <axis xyz="1 0 0" />
-      <limit velocity="6.283" effort="210" lower="-0.785" upper="0.785" />
+      <limit velocity="6.283" effort="210" lower="${-45.*DEG2RAD}" upper="${45.*DEG2RAD}" />
       <dynamics friction="0" damping="3.0"/>
     </joint>
@@ -305,5 +306,5 @@
     <origin xyz="${156.9*mmTom} ${60.*mmTom} ${-108.*mmTom}" rpy="0 0 0" />
     <axis xyz="1 0 0" />
-    <limit velocity="6.283" effort="400" lower="-0.697778" upper="0.87222" />
+    <limit velocity="6.283" effort="400" lower="${-40.*DEG2RAD}" upper="${50.*DEG2RAD}" />
     <dynamics friction="0" damping="3.0"/>
   </joint>
@@ -313,5 +314,5 @@
     <origin xyz="-0.0889 0.121032 -0.217872" rpy="0 0 0" />
     <axis xyz="0 0 1" />
-    <limit velocity="6.283" effort="140" lower="-0.872222" upper="1.57" />
+    <limit velocity="6.283" effort="140" lower="${-50.*DEG2RAD}" upper="${90.*DEG2RAD}" />
     <dynamics friction="0" damping="3.0"/>
   </joint>
@@ -321,5 +322,5 @@
     <origin xyz="0.0 0.0 0.0" rpy="0 0 0" />
     <axis xyz="0 1 0" />
-    <limit velocity="6.283" effort="400" lower="-2.09333" upper="1.046667" />
+    <limit velocity="6.283" effort="400" lower="${-120.*DEG2RAD}" upper="${60.*DEG2RAD}" />
     <dynamics friction="0" damping="3.0"/>
   </joint>
@@ -329,5 +330,5 @@
     <origin xyz="0.0 0.0 -0.356" rpy="0 0 0" />
     <axis xyz="0 1 0" />
-    <limit velocity="6.283" effort="400" lower="0.0" upper="2.442222" />
+    <limit velocity="6.283" effort="400" lower="0.0" upper="${140.*DEG2RAD}" />
     <dynamics friction="0" damping="3.0"/>
   </joint>
@@ -337,5 +338,5 @@
     <origin xyz="0.0 0.0 -0.4" rpy="0 0 0" />
     <axis xyz="0 1 0" />
-    <limit velocity="6.283" effort="330" lower="-1.39556" upper="0.697778" />
+    <limit velocity="6.283" effort="330" lower="${-80.*DEG2RAD}" upper="${40.*DEG2RAD}" />
     <dynamics friction="0" damping="3.0"/>
   </joint>
@@ -345,5 +346,5 @@
     <origin xyz="0.0 0.0 0.0" rpy="0 0 0" />
     <axis xyz="1 0 0" />
-    <limit velocity="6.283" effort="210" lower="-0.785" upper="0.785" />
+    <limit velocity="6.283" effort="210" lower="${-45.*DEG2RAD}" upper="${45.*DEG2RAD}" />
     <dynamics friction="0" damping="3.0"/>
   </joint>

Commit message: change the wall position and add hand pad

File: walkman_urdf/urdf/parts/arms.urdf.xacro (robot description, xacro)
@@ -133,14 +133,18 @@
  </inertial>
  <visual>
-   <origin xyz="0 0 0" rpy="0 0 0"/>
+   <!--origin xyz="0 0 0" rpy="0 0 0"/-->
+   <origin xyz="0 0 0" rpy="0 0 0.785"/>
    <geometry name="RWrMot3_visual">
-     <mesh filename="package://walkman_urdf/meshes/ForearmYaw.STL" scale="0.001 0.001 0.001" />
+     <!--mesh filename="package://walkman_urdf/meshes/ForearmYaw.STL" scale="0.001 0.001 0.001" /-->
+     <box size="0.1 0.1 0.01" />
    </geometry>
   <material name="blue"/>
  </visual>
  <collision>
-   <origin xyz="0 0 0" rpy="0 0 0"/>
+   <!--origin xyz="0 0 0" rpy="0 0 0"/-->
+   <origin xyz="0 0 0" rpy="0 0 0.785"/>
    <geometry name="RWrMot3_collision">
-     <mesh filename="package://walkman_urdf/meshes/simple/ForearmYaw.STL" scale="0.001 0.001 0.001" />
+     <!--mesh filename="package://walkman_urdf/meshes/simple/ForearmYaw.STL" scale="0.001 0.001 0.001" /-->
+     <box size="0.1 0.1 0.01" />
    </geometry>
  </collision>
@@ -330,14 +334,18 @@
  </inertial>
  <visual>
-   <origin xyz="0 0 0" rpy="0 0 0"/>
+   <!--origin xyz="0 0 0" rpy="0 0 0"/-->
+   <origin xyz="0 0 0" rpy="0 0 0.785"/>
    <geometry name="LWrMot3_visual">
-     <mesh filename="package://walkman_urdf/meshes/ForearmYaw.STL" scale="0.001 -0.001 0.001" />
+     <!--mesh filename="package://walkman_urdf/meshes/ForearmYaw.STL" scale="0.001 -0.001 0.001" /-->
+     <box size="0.1 0.1 0.01" />
    </geometry>
   <material name="blue"/>
  </visual>
  <collision>
-   <origin xyz="0 0 0" rpy="0 0 0"/>
+   <!--origin xyz="0 0 0" rpy="0 0 0"/-->
+   <origin xyz="0 0 0" rpy="0 0 0.785"/>
    <geometry name="LWrMot3_collision">
-     <mesh filename="package://walkman_urdf/meshes/simple/ForearmYaw.STL" scale="0.001 -0.001 0.001" />
+     <!--mesh filename="package://walkman_urdf/meshes/simple/ForearmYaw.STL" scale="0.001 -0.001 0.001" /-->
+     <box size="0.1 0.1 0.01" />
    </geometry>
  </collision>

Commit message: Updated arms joint limits

File: walkman_urdf/urdf/parts/arms.urdf.xacro (robot description, xacro)
@@ -151,5 +151,5 @@
     <origin xyz="${45.7475*mmTom} ${-169.137*mmTom} ${155.126*mmTom}" rpy="-0.174533 0 0.5235988" />
     <axis xyz="0 1 0" />
-    <limit velocity="6.283" effort="147" lower="${-195.*DEG2RAD}" upper="${95.*DEG2RAD}" />
+    <limit velocity="6.283" effort="147" lower="-3.359" upper="1.606" />
     <dynamics friction="0" damping="3.0"/>
 </joint>
@@ -159,5 +159,5 @@
     <origin xyz="${-90.15*mmTom} ${-62*mmTom} 0" rpy="0.1745327 0 0" />
     <axis xyz="1 0 0" />
-    <limit velocity="6.283" effort="120" lower="${-200.*DEG2RAD}" upper="0" />
+    <limit velocity="6.283" effort="120" lower="-3.43" upper="-0.004" />
     <dynamics friction="0" damping="3.0"/>
 </joint>
@@ -167,5 +167,5 @@
     <origin xyz="${90.15*mmTom} 0 ${-218.15*mmTom}" rpy="0 0 0" />
     <axis xyz="0 0 1" />
-    <limit velocity="6.283" effort="147" lower="${-150.*DEG2RAD}" upper="${150.*DEG2RAD}" />
+    <limit velocity="6.283" effort="147" lower="-2.55" upper="2.55" />
     <dynamics friction="0" damping="3.0"/>
 </joint>
@@ -175,5 +175,5 @@
     <origin xyz="${45.*mmTom} ${-55.15*mmTom} ${-74.*mmTom}" rpy="0 0 0" />
     <axis xyz="0 1 0" />
-    <limit velocity="6.283" effort="147" lower="${-170.0*toRad}" upper="${34.0*toRad}" />
+    <limit velocity="6.283" effort="147" lower="-2.488" upper="0.292" />
     <dynamics friction="0" damping="3.0"/>
 </joint>
@@ -183,5 +183,5 @@
     <origin xyz="${-15.*mmTom} ${55.15*mmTom} ${-95.*mmTom}" rpy="0 0 0"/>
     <axis xyz="0 0 1" />
-    <limit velocity="6.283" effort="55" lower="${-150*DEG2RAD}" upper="${150*DEG2RAD}" />
+    <limit velocity="6.283" effort="55" lower="-2.55" upper="2.55" />
     <dynamics friction="0" damping="0.03"/>
 </joint>
@@ -191,5 +191,5 @@
     <origin xyz="0 ${-49*mmTom} ${-156.*mmTom}" rpy="0 0 0"/>
     <axis xyz="0 1 0"/>
-    <limit velocity="6.283" effort="55" lower="${-90.*DEG2RAD}" upper="${90.*DEG2RAD}" />
+    <limit velocity="6.283" effort="55" lower="-1.542" upper="1.508" />
     <dynamics friction="0" damping="0.03"/>
 </joint>
@@ -199,5 +199,5 @@
        <origin xyz="0 ${49*mmTom} ${-174.*mmTom}" rpy="0 0 0"/>
        <axis xyz="0 0 1"/>
-       <limit velocity="6.283" effort="27" lower="${-150.*DEG2RAD}" upper="${150.*DEG2RAD}" />
+       <limit velocity="6.283" effort="27" lower="-2.55" upper="2.55" />
        <dynamics friction="0" damping="0.03"/>
 </joint>
@@ -348,5 +348,5 @@
     <origin xyz="${45.7475*mmTom} ${169.137*mmTom} ${155.126*mmTom}" rpy="0.174533 0 -0.5235988" />
     <axis xyz="0 1 0" />
-    <limit velocity="6.283" effort="147" lower="${-195.*DEG2RAD}" upper="${95.*DEG2RAD}" />
+    <limit velocity="6.283" effort="147" lower="-3.352" upper="1.603" />
     <dynamics friction="0" damping="3.0"/>
 </joint>
@@ -356,5 +356,5 @@
     <origin xyz="${-90.15*mmTom} ${62*mmTom} 0" rpy="-0.1745327 0 0" />
     <axis xyz="1 0 0" />
-    <limit velocity="6.283" effort="120" lower="0" upper="${200.*DEG2RAD}" />
+    <limit velocity="6.283" effort="120" lower="0.037" upper="3.517" />
     <dynamics friction="0" damping="3.0"/>
 </joint>
@@ -364,5 +364,5 @@
     <origin xyz="${90.15*mmTom} 0 ${-218.15*mmTom}" rpy="0 0 0" />
     <axis xyz="0 0 1" />
-    <limit velocity="6.283" effort="147" lower="${-150.*DEG2RAD}" upper="${150.*DEG2RAD}" />
+    <limit velocity="6.283" effort="147" lower="-2.55" upper="2.55" />
     <dynamics friction="0" damping="3.0"/>
 </joint>
@@ -372,5 +372,5 @@
     <origin xyz="${45.*mmTom} ${55.15*mmTom} ${-74.*mmTom}" rpy="0 0 0" />
     <axis xyz="0 1 0" />
-    <limit velocity="6.283" effort="147" lower="${-145.0*DEG2RAD}" upper="${20.0*DEG2RAD}" />
+    <limit velocity="6.283" effort="147" lower="-2.492" upper="0.298" />
     <dynamics friction="0" damping="3.0"/>
 </joint>
@@ -380,5 +380,5 @@
     <origin xyz="${-15.*mmTom} ${-55.15*mmTom} ${-95.*mmTom}" rpy="0 0 0"/>
     <axis xyz="0 0 1" />
-    <limit velocity="6.283" effort="55" lower="${-150.0*DEG2RAD}" upper="${150.0*DEG2RAD}" />
+    <limit velocity="6.283" effort="55" lower="-2.55" upper="2.55" />
     <dynamics friction="0" damping="0.03"/>
 </joint>
@@ -388,5 +388,5 @@
     <origin xyz="0 ${49*mmTom} ${-156.*mmTom}" rpy="0 0 0"/>
     <axis xyz="0 1 0"/>
-    <limit velocity="6.283" effort="55" lower="${-90.0*DEG2RAD}" upper="${90.0*DEG2RAD}" />
+    <limit velocity="6.283" effort="55" lower="-1.562" upper="1.478" />
     <dynamics friction="0" damping="0.03"/>
 </joint>
@@ -396,5 +396,5 @@
        <origin xyz="0 ${-49*mmTom} ${-174.*mmTom}" rpy="0 0 0"/>
        <axis xyz="0 0 1"/>
-       <limit velocity="6.283" effort="27" lower="${-150.0*DEG2RAD}" upper="${150.0*DEG2RAD}" />
+       <limit velocity="6.283" effort="27" lower="-2.55" upper="2.55" />
        <dynamics friction="0" damping="0.03"/>
 </joint>

Commit message: modify hand orientation

File: walkman_urdf/urdf/parts/arms.urdf.xacro (robot description, xacro)
@@ -134,5 +134,5 @@
  <visual>
    <!--origin xyz="0 0 0" rpy="0 0 0"/-->
-   <origin xyz="0 0 0" rpy="0 0 0.785"/>
+   <origin xyz="0 0 0" rpy="0 0 0"/>
    <geometry name="RWrMot3_visual">
      <!--mesh filename="package://walkman_urdf/meshes/ForearmYaw.STL" scale="0.001 0.001 0.001" /-->
@@ -143,5 +143,5 @@
  <collision>
    <!--origin xyz="0 0 0" rpy="0 0 0"/-->
-   <origin xyz="0 0 0" rpy="0 0 0.785"/>
+   <origin xyz="0 0 0" rpy="0 0 0"/>
    <geometry name="RWrMot3_collision">
      <!--mesh filename="package://walkman_urdf/meshes/simple/ForearmYaw.STL" scale="0.001 0.001 0.001" /-->
@@ -335,5 +335,5 @@
  <visual>
    <!--origin xyz="0 0 0" rpy="0 0 0"/-->
-   <origin xyz="0 0 0" rpy="0 0 0.785"/>
+   <origin xyz="0 0 0" rpy="0 0 0"/>
    <geometry name="LWrMot3_visual">
      <!--mesh filename="package://walkman_urdf/meshes/ForearmYaw.STL" scale="0.001 -0.001 0.001" /-->
@@ -344,5 +344,5 @@
  <collision>
    <!--origin xyz="0 0 0" rpy="0 0 0"/-->
-   <origin xyz="0 0 0" rpy="0 0 0.785"/>
+   <origin xyz="0 0 0" rpy="0 0 0"/>
    <geometry name="LWrMot3_collision">
      <!--mesh filename="package://walkman_urdf/meshes/simple/ForearmYaw.STL" scale="0.001 -0.001 0.001" /-->
