Commit message: added collision link to L/RSoftHand

File: walkman_urdf/urdf/parts/soft_hand.urdf.xacro (robot description, xacro)
@@ -4,5 +4,12 @@
 <xacro:property name="PI_2" value="1.57079632679" />
 <!-- LINKS -->
-<link name="RSoftHand"/>
+<link name="RSoftHand">
+<collision>
+      <origin xyz="0.0 0.0 0.0" rpy="0.0 0.0 0.0"/>
+      <geometry name="RSoftHand_collision">
+        <box size="0.1 -0.01 0.1" />
+      </geometry>
+    </collision>
+</link>
 <link name="TCP_R"/>
 <link name="RSoftHandLink">
@@ -26,5 +33,12 @@
    </collision>
 </link>
-  <link name="LSoftHand"/>
+  <link name="LSoftHand">
+    <collision>
+      <origin xyz="0.0 0.0 0.0" rpy="0.0 0.0 0.0"/>
+      <geometry name="LSoftHand_collision">
+        <box size="0.1 0.01 0.1" />
+      </geometry>
+    </collision>
+  </link>
   <link name="TCP_L"/>
 <link name="LSoftHandLink">

Commit message: Added dynamics for R/LSoftHand

File: walkman_urdf/urdf/parts/soft_hand.urdf.xacro (robot description, xacro)
@@ -5,5 +5,10 @@
 <!-- LINKS -->
 <link name="RSoftHand">
-<collision>
+    <inertial>
+      <origin xyz="0.0 0.0 0.0" rpy="0 0 0"/>
+      <mass value="0.001"/>
+      <inertia ixx="1e-12"  ixy="0.0"  ixz="0.0" iyy="1e-12" iyz="0.0" izz="1e-12" />
+    </inertial>
+    <collision>
       <origin xyz="0.0 0.0 0.0" rpy="0.0 0.0 0.0"/>
       <geometry name="RSoftHand_collision">
@@ -34,4 +39,9 @@
 </link>
   <link name="LSoftHand">
+    <inertial>
+      <origin xyz="0.0 0.0 0.0" rpy="0 0 0"/>
+      <mass value="0.001"/>
+      <inertia ixx="1e-12"  ixy="0.0"  ixz="0.0" iyy="1e-12" iyz="0.0" izz="1e-12" />
+    </inertial>
     <collision>
       <origin xyz="0.0 0.0 0.0" rpy="0.0 0.0 0.0"/>
