Commit message: Added interface between arm and hands (wrist)

File: walkman_urdf/urdf/walkman.urdf.xacro (robot description, xacro)
@@ -33,22 +33,4 @@
 </joint>
 <!--
-	<link name="l_arm_ft"/>
-	<link name="r_arm_ft"/>
-	<joint name="l_arm_ft_joint" type="fixed">
-	    <parent link="LWrMot3"/>
-	    <child link="l_arm_ft"/>
-	    <origin xyz="0 0 -0.0565" rpy="0 0 0" />
-	</joint>
-	<joint name="r_arm_ft_joint" type="fixed">
-	    <parent link="RWrMot3"/>
-	    <child link="r_arm_ft"/>
-	    <origin xyz="0 0 -0.0565" rpy="0 0 0" />
-	</joint>
-	<link name="l_wrist"/>
-	<link name="r_wrist"/>
-	<xacro:include filename="$(find bigman_urdf)/urdf/parts/forearms.urdf.xacro" />
-       <xacro:if value="${BIGMAN_ADD_RAISING_SUPPORT}">
-	       <xacro:include filename="$(find bigman_urdf)/urdf/parts/forearm_reference_frame.urdf.xacro" />
-       </xacro:if>
 	<xacro:include filename="$(find bigman_urdf)/urdf/parts/soft_hand.urdf.xacro" />
 -->

File: walkman_urdf/urdf/walkman_base.urdf.xacro (robot description, xacro)
@@ -10,4 +10,5 @@
 <xacro:property name="mm2Tom2" value="${0.001*0.001}" />
 <xacro:property name="tonsToKg" value="1000.0" />
+<xacro:property name="PI" value="3.14159265359" />
 <!--
 The coordinate frame called base_link is rigidly attached to the robot root body. It is recommended to choose the robot waist as its root body. The base_link can be attached to the root in any arbitrary position or orientation; for every hardware platform there will be a different place on the base that provides an obvious point of reference. Note that REP 103 [1] specifies a preferred orientation for frames. -->
@@ -68,6 +69,44 @@
 <xacro:include filename="$(find walkman_urdf)/urdf/parts/neck.urdf.xacro" />
 <xacro:include filename="$(find walkman_urdf)/urdf/parts/arms.urdf.xacro" />
-<link name="l_wrist"/>
-<link name="r_wrist"/>
+<link name="l_wrist">
+    <inertial>
+      <origin xyz="${8.2161929e-02*mmTom} ${2.6334189*mmTom} ${-1.6465877e+01*mmTom}" rpy="0 0 0"/>
+      <mass value="3.7827821e-01"/>
+      <inertia ixx="${2.3321716e+02*mm2Tom2}"  ixy="${2.3681435*mm2Tom2}"  ixz="${-1.8039102*mm2Tom2}" iyy="${2.0626291e+02*mm2Tom2}" iyz="${3.1588290e+01*mm2Tom2}" izz="${2.7399881e+02*mm2Tom2}" />
+    </inertial>
+    <visual>
+      <origin xyz="0 0 0" rpy="${PI} 0 0"/>
+      <geometry name="LShp_visual">
+        <mesh filename="package://walkman_urdf/meshes/Wrist.STL" scale="0.001 -0.001 0.001" />
+      </geometry>
+      <material name="dark_grey"/>
+    </visual>
+    <collision>
+      <origin xyz="0 0 0" rpy="${PI} 0 0"/>
+      <geometry name="LShp_collision">
+        <mesh filename="package://walkman_urdf/meshes/simple/Wrist.STL" scale="0.001 -0.001 0.001" />
+      </geometry>
+    </collision>
+</link>
+<link name="r_wrist">
+    <inertial>
+      <origin xyz="${8.2161929e-02*mmTom} ${-2.6334189*mmTom} ${-1.6465877e+01*mmTom}" rpy="0 0 0"/>
+      <mass value="3.7827821e-01"/>
+      <inertia ixx="${2.3321716e+02*mm2Tom2}"  ixy="${-2.3681435*mm2Tom2}"  ixz="${-1.8039102*mm2Tom2}" iyy="${2.0626291e+02*mm2Tom2}" iyz="${-3.1588290e+01*mm2Tom2}" izz="${2.7399881e+02*mm2Tom2}" />
+    </inertial>
+    <visual>
+      <origin xyz="0 0 0" rpy="${PI} 0 0"/>
+      <geometry name="RShp_visual">
+        <mesh filename="package://walkman_urdf/meshes/Wrist.STL" scale="0.001 0.001 0.001" />
+      </geometry>
+      <material name="dark_grey"/>
+    </visual>
+    <collision>
+      <origin xyz="0 0 0" rpy="${PI} 0 0"/>
+      <geometry name="RShp_collision">
+        <mesh filename="package://walkman_urdf/meshes/simple/Wrist.STL" scale="0.001 0.001 0.001" />
+      </geometry>
+    </collision>
+</link>
 <joint name="l_wrist_joint" type="fixed">
        <parent link="LWrMot3"/>
@@ -80,3 +119,17 @@
        <origin xyz="0 0 0" rpy="0 0 0" />
 </joint>
+<!--
+<link name="l_arm_ft"/>
+	<link name="r_arm_ft"/>
+	<joint name="l_arm_ft_joint" type="fixed">
+	    <parent link="LWrMot3"/>
+	    <child link="l_arm_ft"/>
+	    <origin xyz="0 0 -0.0565" rpy="0 0 0" />
+	</joint>
+	<joint name="r_arm_ft_joint" type="fixed">
+	    <parent link="RWrMot3"/>
+	    <child link="r_arm_ft"/>
+	    <origin xyz="0 0 -0.0565" rpy="0 0 0" />
+	</joint>
+-->
 </robot>
