Commit message: added gaze frame in the middle of the neck pitch joint (probably we are going to move it)

File: walkman_urdf/urdf/walkman_base.urdf.xacro (robot description, xacro)
@@ -68,4 +68,10 @@
 <xacro:include filename="$(find walkman_urdf)/urdf/parts/torso.urdf.xacro" />
 <xacro:include filename="$(find walkman_urdf)/urdf/parts/neck.urdf.xacro" />
+<link name="gaze"/>
+<joint name="gaze_joint" type="fixed">
+       <parent link="NeckPitch"/>
+       <child link="gaze"/>
+       <origin xyz="0 ${-34.25*mmTom} 0" rpy="0 0 0" />
+</joint>
 <xacro:include filename="$(find walkman_urdf)/urdf/parts/arms.urdf.xacro" />
 <link name="l_wrist">
