Commit message: Updated position of IMU (doc and xacro)

File: walkman_urdf/urdf/sensors/imu.urdf.xacro (robot description, xacro)
@@ -2,4 +2,5 @@
 <robot xmlns:xacro="http://ros.org/wiki/xacro">
 <xacro:property name="PI" value="3.14159265359" />
+<xacro:property name="mmTom" value="0.001" />
 <link name="imu_link">
     <inertial>
@@ -19,5 +20,5 @@
     <parent link="Waist"/>
     <child link="imu_link"/>
-    <origin xyz="0.0 0.0 0.0" rpy="0 0 0"/>
+    <origin xyz="${116.998*mmTom} ${0.0283129*mmTom} ${-47.8857*mmTom}" rpy="0 0 0"/>
 </joint>
 </robot>

Commit message: Updated IMU and doc

File: walkman_urdf/urdf/sensors/imu.urdf.xacro (robot description, xacro)
@@ -16,9 +16,8 @@
     </visual>
   </link>
-<!-- TODO: CHANGE THE ORIGIN OF THE SENSOR ACCORDING TO THE REAL ONE -->
 <joint name="imu_joint" type="fixed">
     <parent link="Waist"/>
     <child link="imu_link"/>
-    <origin xyz="${116.998*mmTom} ${0.0283129*mmTom} ${-47.8857*mmTom}" rpy="0 0 0"/>
+    <origin xyz="${117.0*mmTom} 0.0 ${-47.7493*mmTom}" rpy="0 0 0"/>
 </joint>
 </robot>
