Commit message: added wrist frames and arms to urdf

File: walkman_srdf/srdf/walkman.srdf.xacro (robot description, xacro)
@@ -28,4 +28,10 @@
         <chain base_link="Waist" tip_link="DWYTorso"/>
     </group>
+   <group name="left_arm">
+        <chain base_link="DWYTorso" tip_link="l_wrist"/>
+    </group>
+    <group name="right_arm">
+        <chain base_link="DWYTorso" tip_link="r_wrist"/>
+    </group>
    <group name="head">
         <chain base_link="DWYTorso" tip_link="NeckPitch"/>
@@ -35,4 +41,6 @@
         <group name="right_leg"/>
         <group name="torso"/>
+        <group name="left_arm"/>
+        <group name="right_arm"/>
         <group name="head"/>
     </group>

File: walkman_urdf/urdf/walkman_base.urdf.xacro (robot description, xacro)
@@ -68,3 +68,15 @@
 <xacro:include filename="$(find walkman_urdf)/urdf/parts/neck.urdf.xacro" />
 <xacro:include filename="$(find walkman_urdf)/urdf/parts/arms.urdf.xacro" />
+<link name="l_wrist"/>
+<link name="r_wrist"/>
+<joint name="l_wrist_joint" type="fixed">
+       <parent link="LWrMot3"/>
+       <child link="l_wrist"/>
+       <origin xyz="0 0 0" rpy="0 0 0" />
+</joint>
+<joint name="r_wrist_joint" type="fixed">
+       <parent link="RWrMot3"/>
+       <child link="r_wrist"/>
+       <origin xyz="0 0 0" rpy="0 0 0" />
+</joint>
 </robot>

Commit message: Added imu. Frame needs to be updated

File: walkman_srdf/srdf/walkman.srdf.xacro (robot description, xacro)
@@ -18,4 +18,7 @@
          <joint name="l_leg_ft_joint"/>
 	  <joint name="r_leg_ft_joint"/>
+    </group>
+    <group name="imu_sensors">
+         <link name="imu_link"/>
     </group>
     <group name="left_leg">

File: walkman_urdf/urdf/gazebo/microstrain_3dmgx2_imu.gazebo.xacro (robot description, xacro)
@@ -33,30 +33,3 @@
         </sensor>
        </gazebo>
-       <gazebo reference="imu_link2">
-        <sensor name="imu_link2" type="imu">
-         <always_on>1</always_on>
-         <update_rate>1000</update_rate>
-         <visualize>true</visualize>
-         <topic>__default_topic__</topic>
-	 <imu>
-          <!--
-          <noise>
-           <type>gaussian</type>
-            <rate>
-             <mean>0.0</mean>
-             <stddev>2e-4</stddev>
-             <bias_mean>0.0000075</bias_mean>
-             <bias_stddev>0.0000008</bias_stddev>
-            </rate>
-            <accel>
-             <mean>0.0</mean>
-             <stddev>1.7e-2</stddev>
-             <bias_mean>0.1</bias_mean>
-             <bias_stddev>0.001</bias_stddev>
-            </accel>
-          </noise>
-          -->
-         </imu>
-        </sensor>
-       </gazebo>
 </robot>

File: walkman_urdf/urdf/sensors/imu.urdf.xacro (robot description, xacro)
@@ -15,26 +15,9 @@
     </visual>
   </link>
-<link name="imu_link2">
-    <inertial>
-      <mass value="0.01"/>
-      <origin xyz="0 0 0"/>
-      <inertia ixx="1.0E-6" ixy="0" ixz="0" iyy="1.0E-6" iyz="0" izz="1.0E-6"/>
-    </inertial>
-    <visual>
-      <origin rpy="0 0 0" xyz="0 0 0"/>
-      <geometry>
-        <box size="0.01 0.01 0.01"/>
-      </geometry>
-    </visual>
-  </link>
+<!-- TODO: CHANGE THE ORIGIN OF THE SENSOR ACCORDING TO THE REAL ONE -->
 <joint name="imu_joint" type="fixed">
     <parent link="Waist"/>
     <child link="imu_link"/>
-    <origin xyz="0.0535 0.0 0.0601" rpy="0 0 0"/>
-</joint>
-<joint name="imu_joint2" type="fixed">
-    <parent link="Waist"/>
-    <child link="imu_link2"/>
-    <origin xyz="0.0135 0.0 0.0601" rpy="0 0 0"/>
+    <origin xyz="0.0 0.0 0.0" rpy="0 0 0"/>
 </joint>
 </robot>

File: walkman_urdf/urdf/walkman.urdf.xacro (robot description, xacro)
@@ -52,5 +52,5 @@
        </xacro:if>
 	<xacro:include filename="$(find bigman_urdf)/urdf/parts/soft_hand.urdf.xacro" />
-<xacro:include filename="$(find bigman_urdf)/urdf/sensors/imu.urdf.xacro"/>
 -->
+<xacro:include filename="$(find walkman_urdf)/urdf/sensors/imu.urdf.xacro"/>
 </robot>

Commit message: added arms ft in srdf

File: walkman_srdf/srdf/walkman.srdf.xacro (robot description, xacro)
@@ -17,5 +17,7 @@
     <group name="force_torque_sensors">
          <joint name="l_leg_ft_joint"/>
-	  <joint name="r_leg_ft_joint"/>
+	 <joint name="r_leg_ft_joint"/>
+         <joint name="l_arm_ft_joint"/>
+	 <joint name="r_arm_ft_joint"/>
     </group>
     <group name="imu_sensors">

Commit message: Updated model for the magnetic grasp

File: walkman_srdf/srdf/walkman.srdf.xacro (robot description, xacro)
@@ -23,4 +23,8 @@
     <group name="imu_sensors">
          <link name="imu_link"/>
+    </group>
+    <group name="hands">
+      <joint name="r_wrist_joint"/>
+      <joint name="l_wrist_joint"/>
     </group>
     <group name="left_leg">
@@ -50,3 +54,34 @@
         <group name="head"/>
     </group>
+    <group_state group="chains" name="home">
+        <joint name="NeckYawj" value="0.0"/>
+        <joint name="NeckPitchj" value="0.6"/>
+        <joint name="WaistYaw" value="0.0"/>
+        <joint name="RShSag" value="1.10"/>
+        <joint name="RShLat" value="-0.20"/>
+        <joint name="RShYaw" value="-1.50"/>
+        <joint name="RElbj" value="-2.0"/>
+        <joint name="RForearmPlate" value="0"/>
+        <joint name="RWrj1" value="-0.0"/>
+        <joint name="RWrj2" value="-0.0"/>
+        <joint name="LShSag" value="1.10"/>
+        <joint name="LShLat" value="0.20"/>
+        <joint name="LShYaw" value="1.5"/>
+        <joint name="LElbj" value="-2.0"/>
+        <joint name="LForearmPlate" value="0"/>
+        <joint name="LWrj1" value="0.0"/>
+        <joint name="LWrj2" value="-0.0"/>
+        <joint name="RHipLat" value="0.06"/>
+        <joint name="RHipYaw" value="0.0"/>
+        <joint name="RHipSag" value="-0.45"/>
+        <joint name="RKneeSag" value="0.90"/>
+        <joint name="RAnkSag" value="-0.45"/>
+        <joint name="RAnkLat" value="-0.06"/>
+        <joint name="LHipLat" value="-0.06"/>
+        <joint name="LHipYaw" value="0.0"/>
+        <joint name="LHipSag" value="-0.45"/>
+        <joint name="LKneeSag" value="0.90"/>
+        <joint name="LAnkSag" value="-0.45"/>
+        <joint name="LAnkLat" value="0.06"/>
+    </group_state>
 </robot>

File: walkman_urdf/urdf/gazebo/magnetic_attach_ros.gazebo.xacro (robot description, xacro)
@@ -3,8 +3,8 @@
 <gazebo>
 <plugin name="magnetic_LSoftHand" filename="libmagnetic.so">
-       <link_name>LSoftHand</link_name>
+       <link_name>LWrMot3</link_name>
 </plugin>
 <plugin name="magnetic_RSoftHand" filename="libmagnetic.so">
-       <link_name>RSoftHand</link_name>
+       <link_name>RWrMot3</link_name>
 </plugin>
 </gazebo>

File: walkman_urdf/urdf/parts/soft_hand.urdf.xacro (robot description, xacro)
@@ -4,17 +4,5 @@
 <xacro:property name="PI_2" value="1.57079632679" />
 <!-- LINKS -->
-<link name="RSoftHand">
-    <inertial>
-      <origin xyz="0.0 0.0 0.0" rpy="0 0 0"/>
-      <mass value="0.001"/>
-      <inertia ixx="1e-12"  ixy="0.0"  ixz="0.0" iyy="1e-12" iyz="0.0" izz="1e-12" />
-    </inertial>
-    <collision>
-      <origin xyz="0.0 0.0 0.0" rpy="0.0 0.0 0.0"/>
-      <geometry name="RSoftHand_collision">
-        <box size="0.1 -0.01 0.1" />
-      </geometry>
-    </collision>
-</link>
+<link name="RSoftHand"/>
 <link name="TCP_R"/>
 <link name="RSoftHandLink">
@@ -38,17 +26,5 @@
    </collision>
 </link>
-  <link name="LSoftHand">
-    <inertial>
-      <origin xyz="0.0 0.0 0.0" rpy="0 0 0"/>
-      <mass value="0.001"/>
-      <inertia ixx="1e-12"  ixy="0.0"  ixz="0.0" iyy="1e-12" iyz="0.0" izz="1e-12" />
-    </inertial>
-    <collision>
-      <origin xyz="0.0 0.0 0.0" rpy="0.0 0.0 0.0"/>
-      <geometry name="LSoftHand_collision">
-        <box size="0.1 0.01 0.1" />
-      </geometry>
-    </collision>
-  </link>
+  <link name="LSoftHand"/>
   <link name="TCP_L"/>
 <link name="LSoftHandLink">

Commit message: add force torque sensors in hands

File: walkman_srdf/srdf/walkman.srdf.xacro (robot description, xacro)
@@ -18,4 +18,6 @@
          <joint name="l_leg_ft_joint"/>
 	  <joint name="r_leg_ft_joint"/>
+         <joint name="l_arm_ft_joint"/>
+	 <joint name="r_arm_ft_joint"/>
     </group>
     <group name="left_leg">

File: walkman_urdf/urdf/walkman.urdf.xacro (robot description, xacro)
@@ -32,5 +32,4 @@
     <origin xyz="0.005 0 -0.107" rpy="0 0 0"/>
 </joint>
-<!--
 	<link name="l_arm_ft"/>
 	<link name="r_arm_ft"/>
@@ -45,4 +44,5 @@
 	    <origin xyz="0 0 -0.0565" rpy="0 0 0" />
 	</joint>
+<!--
 	<link name="l_wrist"/>
 	<link name="r_wrist"/>
